File: kicad/_autosave-opamp-front.kicad_pcb (KiCad board)
At the start: 2 copper layers, 87.6 x 118.9 mm, 91 parts, among them J1 B+, J2 SPK, J3 INPUT, J4 GND, J5 B-, J6 GND, Q1 2N5551, Q10 2N2906, Q11 MJL3281C, Q12 2N2904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

Commit message: Moved things a bit
Parts:
- R18, R19: value 1k -> 100
- R20, R21: value 4.7k -> 1.5k
- moved D11 2.54 mm to (65.2, 81.3)
- moved R18 2.54 mm to (68.6, 72.6)
- moved Q5 1.87 mm to (77.4, 79.5)
- moved REF** 1.87 mm to (79.7, 75.2)
- moved D10 1.78 mm to (134.9, 71.4)
- moved R19 1.78 mm to (131.6, 72.9)
- moved REF** 1.52 mm to (121.7, 75.2)
- moved Q9 1.51 mm to (119.4, 79.5)
Routing:
- net Net-(Q11-B): track 87.4 -> 90.1 mm
- net Net-(D13-A): track 120.2 -> 121.6 mm
- net Net-(Q13-B): track 63.7 -> 65.1 mm
- net Net-(Q7-B): track 35.4 -> 36.7 mm
- net /B-: track 79.4 -> 78.3 mm
- net Net-(Q11-E): track 39.4 -> 40.5 mm
- net Net-(Q8-B): track 31.9 -> 32.6 mm
- net Net-(Q13-E): track 34.1 -> 34.9 mm
- net /B+: track 84.5 -> 85.2 mm
- net Net-(D14-K): track 125.6 -> 126.2 mm
Other:
- board text added: "https://github.com/prydin/opamp-frontend-class-ab"
