File: kicad/_autosave-opamp-front.kicad_sch (KiCad schematic)
At the start: 84 parts, among them J1 B+, J2 SPK, J3 INPUT, J4 GND, J5 B-, J6 GND, Q1 2N5551, Q10 2N2906, Q11 MJL3281C, Q12 2N2904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

Commit message: Moved things a bit
Parts:
- R18, R19: value 1k -> 100
- R20, R21: value 4.7k -> 1.5k
Changed lines of the file:
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@@
 			)
 		)
-		(property "Value" "4.7k"
+		(property "Value" "1.5k"
 			(at 190.5 60.7059 0)
 			(effects
@@
 			)
 		)
-		(property "Value" "1k"
+		(property "Value" "100"
 			(at 219.71 91.44 90)
 			(effects
@@
 			)
 		)
-		(property "Value" "4.7k"
+		(property "Value" "1.5k"
 			(at 190.5 102.6159 0)
 			(effects
@@
 			)
 		)
-		(property "Value" "1k"
+		(property "Value" "100"
 			(at 219.71 60.96 90)
 			(effects
