File: kicad/opamp-front.kicad_pcb (KiCad board)
At the start: 2 copper layers, 101.3 x 102.4 mm, 91 parts, among them J1 INPUT, J2 GND, J3 SPK, J4 GND, J5 B+, J6 B-, Q1 BD140, Q10 BD139, Q11 BD139, Q12 BD140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

Commit message: Release candidate 1
Parts:
- added C17: 220p, Capacitor_THT:C_Rect_L7.2mm_W3.0mm_P5.00mm_FKS2_FKP2_MKS2_MKP2, F.Cu at (133.9, 127.5)
- added R31: 10, Custom:R_Axial_DIN0204_L3.6mm_D1.6mm_P7.62mm_Horizontal_HandSolder, F.Cu at (90.2, 113.0)
- R1, R10, R12, R13, R14, R15, R16, R17, R19, R2, R22, R23, R24, R25, R26, R27, R29, R3, R30, R4, R7: footprint Resistor_THT:R_Axial_DIN0204_L3.6mm_D1.6mm_P7.62mm_Horizontal -> Custom:R_Axial_DIN0204_L3.6mm_D1.6mm_P7.62mm_Horizontal_HandSolder
- R11: value 1k -> 680; footprint Resistor_THT:R_Axial_DIN0204_L3.6mm_D1.6mm_P7.62mm_Horizontal -> Custom:R_Axial_DIN0204_L3.6mm_D1.6mm_P7.62mm_Horizontal_HandSolder
- R18, R28: value 0.22 -> 0.22 3W
- R20, R21: value 10 -> 10 3W
- R5, R8: value 10k -> 6.8k; footprint Resistor_THT:R_Axial_DIN0204_L3.6mm_D1.6mm_P7.62mm_Horizontal -> Custom:R_Axial_DIN0204_L3.6mm_D1.6mm_P7.62mm_Horizontal_HandSolder
- R6, R9: value 4.7k -> 680; footprint Resistor_THT:R_Axial_DIN0204_L3.6mm_D1.6mm_P7.62mm_Horizontal -> Custom:R_Axial_DIN0204_L3.6mm_D1.6mm_P7.62mm_Horizontal_HandSolder
- moved D6 5.84 mm to (78.0, 113.1)
- moved D7 5.84 mm to (84.3, 105.5)
- moved D5 5.84 mm to (64.9, 113.1)
- moved R5 5.84 mm to (71.3, 113.0)
- moved R6 5.84 mm to (58.4, 105.4)
- moved Q4 1.27 mm to (103.4, 97.8)
- moved C14 1.08 mm to (85.6, 47.5)
- moved RV1 0.76 mm to (109.0, 53.6)
- moved R8 0.21 mm to (109.2, 105.4)
- moved D4 0.10 mm to (102.4, 105.5)
- moved D8 0.10 mm to (96.0, 113.1)
Connections:
- C1 pad 2: Net-(D7-K) -> Net-(C1-Pad2)
- U1 pad 1: Net-(D7-K) -> Net-(C1-Pad2)
Routing:
- net Net-(D7-K): track 36.9 -> 11.6 mm
- net Net-(C1-Pad2): track 0.00 -> 21.7 mm
- net Net-(R26-Pad2): track 28.6 -> 32.0 mm
- net Net-(Q12-E): track 60.1 -> 63.2 mm
- net Net-(D6-A): track 27.1 -> 30.2 mm
- net /B-: track 96.2 -> 98.6 mm
- net Net-(Q2-E): track 48.0 -> 45.7 mm
- net +15V: track 31.5 -> 33.1 mm
- net Net-(Q13-E): track 51.8 -> 53.2 mm
- net Net-(Q5-E): track 11.1 -> 12.4 mm
- net Net-(D9-A): track 49.3 -> 48.0 mm
- net Net-(Q4-E): track 14.2 -> 15.4 mm
- net Net-(D14-K): track 177.5 -> 178.7 mm
- net Net-(D16-K): track 93.8 -> 95.0 mm
- net Net-(Q8-E): track 73.8 -> 74.9 mm
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Other:
- board text added: "B+"
- board text added: "B-"
- board text added: "SPEAKER"
- board text added: "The TeamworkAmp diyaudio.com"
- board text removed: "SPK"
