File: kicad/opamp-front.kicad_sch (KiCad schematic)
At the start: 84 parts, among them J1 B+, J2 SPK, J3 INPUT, J4 GND, J5 B-, J6 GND, Q1 2N5551, Q10 2N2906, Q11 MJL3281C, Q12 2N2904, Q13 MJL1302C, Q2 BD139, Q3 BD140, Q4 BD139, Q5 BD139, Q6 2N5401, Q7 2N5551, Q8 2N5401, Q9 BD140, U1 LM4562

Commit message: Gerbers generated
Parts:
- added R29: 470, Resistor_THT:R_Axial_DIN0204_L3.6mm_D1.6mm_P7.62mm_Horizontal, symbol Device:R
- added unit 2 of U1
- R16: renamed from R18; value 1k -> 100
- R19: renamed from R20; value 4.7k -> 1.5k
- R23: renamed from R21; value 4.7k -> 1.5k
- R24: renamed from R19; value 1k -> 100
- renumbered C3 to C1, C13 to C10, C9 to C11, C8 to C12, C16 to C13, C6 to C14, C5 to C15, C17 to C16, C15 to C2, C14 to C3, C1 to C4, C2 to C5, C10 to C6, C4 to C7, C12 to C8, C7 to C9, D2 to D1, D7 to D10, D13 to D11, D11 to D12, D15 to D13, D18 to D14, D16 to D15, D14 to D16, D10 to D18, D1 to D2, D9 to D3, D12 to D4, D6 to D5, D4 to D6, D3 to D7, D5 to D8, D8 to D9, J3 to J1, J6 to J2, J2 to J3, J1 to J5, J5 to J6, Q3 to Q1, Q5 to Q10, Q4 to Q11, Q9 to Q12, Q10 to Q2, Q7 to Q3, Q6 to Q4, Q1 to Q5, Q8 to Q6, Q2 to Q7, Q12 to Q8, Q11 to Q9, R5 to R10, R6 to R11, R34 to R12, R2 to R13, R13 to R14, R12 to R15, R33 to R17, R23 to R18, R14 to R2, R31 to R20, R30 to R21, R32 to R22, R17 to R25, R15 to R26, R16 to R27, R25 to R28, R11 to R3, R3 to R4, R7 to R5, R8 to R6, R4 to R7, R9 to R8, R10 to R9
Connections:
- net GND: now also U1.5 (+)
- net at C1.1, C5.1, R1.1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: now also R29.2; no longer C4.2
- new net: C4.2, R29.1
- new net: U1.6 (-), U1.7
Other:
- moved on the sheet: C5, R1

Commit message: WIP
Parts:
- added R30: 10, Resistor_THT:R_Axial_DIN0204_L3.6mm_D1.6mm_P7.62mm_Horizontal, symbol Device:R
Connections:
- net GND: now also R30.2
- net GNDA: now also R30.1
- net at C5.1, R1.1, R29.2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: no longer C1.1
- net at C6.1, R12.1, R13.1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: now also C1.1
Other:
- note added: "Optional Can be left open or shorted"

Commit message: Preparing for public release
Parts:
- Q2: value 2N2906 -> 2N3906
- Q8: value 2N2904 -> 2N3904
- R6, R9: value 4.7k -> 820
Connections:
- net B+: now also D12.1 (K); no longer D12.2 (A)
- net B-: now also D18.2 (A); no longer D18.1 (K)
- net GND: now also D12.2 (A), D18.1 (K); no longer D12.1 (K), D18.2 (A)
Changed lines of the file:
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@@
 			)
 		)
-		(property "Value" "2N2904"
+		(property "Value" "2N3904"
 			(at 129.54 121.9199 0)
 			(effects
@@
 			)
 		)
-		(property "Value" "4.7k"
+		(property "Value" "820"
 			(at 90.17 126.9999 0)
 			(effects
@@
 		(lib_id "Diode:1N4004")
 		(at 198.12 21.59 270)
+		(mirror x)
 		(unit 1)
 		(exclude_from_sim no)
@@
 		(on_board yes)
 		(dnp no)
-		(fields_autoplaced yes)
 		(property "Reference" "D12"
-			(at 200.66 20.3199 90)
+			(at 200.66 22.8601 90)
 			(effects
 				(font
@@
 		)
 		(property "Value" "1N4004"
-			(at 200.66 22.8599 90)
+			(at 200.66 20.3201 90)
 			(effects
 				(font
@@
 			)
 		)
-		(property "Value" "2N2906"
+		(property "Value" "2N3906"
 			(at 129.54 38.0999 0)
 			(effects
@@
 		(lib_id "Diode:1N4004")
 		(at 198.12 135.89 90)
-		(mirror x)
 		(unit 1)
 		(exclude_from_sim no)
@@
 		(dnp no)
 		(property "Reference" "D18"
-			(at 200.66 137.1601 90)
+			(at 200.66 134.6199 90)
 			(effects
 				(font
@@
 		)
 		(property "Value" "1N4004"
-			(at 200.66 134.6201 90)
+			(at 200.66 137.1599 90)
 			(effects
 				(font
@@
 			)
 		)
-		(property "Value" "4.7k"
+		(property "Value" "820"
 			(at 90.17 34.2899 0)
 			(effects

Commit message: Release candidate 1
Parts:
- added C17: 220p, Capacitor_THT:C_Rect_L7.2mm_W3.0mm_P5.00mm_FKS2_FKP2_MKS2_MKP2, symbol Device:C
- added R31: 10, Custom:R_Axial_DIN0204_L3.6mm_D1.6mm_P7.62mm_Horizontal_HandSolder, symbol Device:R
- R1, R10, R12, R13, R14, R15, R16, R17, R19, R2, R22, R23, R24, R25, R29, R3, R30, R4, R7: footprint Resistor_THT:R_Axial_DIN0204_L3.6mm_D1.6mm_P7.62mm_Horizontal -> Custom:R_Axial_DIN0204_L3.6mm_D1.6mm_P7.62mm_Horizontal_HandSolder
- R11: value 1k -> 680; footprint Resistor_THT:R_Axial_DIN0204_L3.6mm_D1.6mm_P7.62mm_Horizontal -> Custom:R_Axial_DIN0204_L3.6mm_D1.6mm_P7.62mm_Horizontal_HandSolder
- R18, R28: value 0.22 -> 0.22 3W
- R20, R21: value 10 -> 10 3W
- R26: value 1k -> 470; footprint Resistor_THT:R_Axial_DIN0204_L3.6mm_D1.6mm_P7.62mm_Horizontal -> Custom:R_Axial_DIN0204_L3.6mm_D1.6mm_P7.62mm_Horizontal_HandSolder
- R27: value 2.7k -> 1.8k; footprint Resistor_THT:R_Axial_DIN0204_L3.6mm_D1.6mm_P7.62mm_Horizontal -> Custom:R_Axial_DIN0204_L3.6mm_D1.6mm_P7.62mm_Horizontal_HandSolder
- R5, R8: value 10k -> 6.8k; footprint Resistor_THT:R_Axial_DIN0204_L3.6mm_D1.6mm_P7.62mm_Horizontal -> Custom:R_Axial_DIN0204_L3.6mm_D1.6mm_P7.62mm_Horizontal_HandSolder
- R6, R9: value 820 -> 680; footprint Resistor_THT:R_Axial_DIN0204_L3.6mm_D1.6mm_P7.62mm_Horizontal -> Custom:R_Axial_DIN0204_L3.6mm_D1.6mm_P7.62mm_Horizontal_HandSolder
- RV1: value 2k -> 500
Connections:
- net GND: now also C17.2
- net GNDA: now also C17.1
- net at D7.1 (K), D8.2 (A): now also R31.2; no longer C1.2, U1.1
- new net: C1.2, R31.1, U1.1
Other:
- note added: "+40V"
- note added: "-40V"
- note added: "All resistors are 1/4W unless otherwise noted."
- note added: "L1 is made by winding 16AWG magnet wire around R20"
- note removed: "Optional Can be left open or shorted"
- moved on the sheet: C1, C2, C3, C4, C5, C7, D1, D2, J1, R1, R13, R29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
