File: kicad/power_supply/power_supply.kicad_pcb (KiCad board)
At the start: 2 copper layers, 129 x 83.3 mm, 24 parts, among them J1 AC1, J2 GND, J3 CT, J4 AC2, J5 V-, J6 V+, J7 GND

Commit message: Preparing for public release
Parts:
- added C13: 4700u, Capacitor_THT:CP_Radial_D18.0mm_P7.50mm, F.Cu at (114.3, 59.2)
- added C14: 4700u, Capacitor_THT:CP_Radial_D18.0mm_P7.50mm, F.Cu at (114.3, 121.1)
- added H1: MountingHole, MountingHole:MountingHole_3.2mm_M3, F.Cu at (66.0, 48.8)
- added H2: MountingHole, MountingHole:MountingHole_3.2mm_M3, F.Cu at (188.2, 48.8)
- added H3: MountingHole, MountingHole:MountingHole_3.2mm_M3, F.Cu at (66.3, 124.5)
- added H4: MountingHole, MountingHole:MountingHole_3.2mm_M3, F.Cu at (188.0, 124.5)
- added Q1: TIP147, Package_TO_SOT_THT:TO-247-3_Horizontal_TabDown, F.Cu at (170.1, 58.0)
- added Q2: TIP142, Package_TO_SOT_THT:TO-247-3_Horizontal_TabDown, F.Cu at (181.0, 115.5)
- added R1: 22, Resistor_THT:R_Axial_DIN0204_L3.6mm_D1.6mm_P7.62mm_Horizontal, F.Cu at (164.3, 61.2)
- added R2: 150, Resistor_THT:R_Axial_DIN0204_L3.6mm_D1.6mm_P7.62mm_Horizontal, F.Cu at (156.0, 53.3)
- added R3: 22, Resistor_THT:R_Axial_DIN0204_L3.6mm_D1.6mm_P7.62mm_Horizontal, F.Cu at (166.1, 112.5)
- added R4: 150, Resistor_THT:R_Axial_DIN0204_L3.6mm_D1.6mm_P7.62mm_Horizontal, F.Cu at (156.2, 120.1)
- added RV1: 2k, Custom:TRIM_T93YA103KT20, F.Cu at (150.9, 57.1)
- added RV2: 2k, Custom:TRIM_T93YA103KT20, F.Cu at (151.4, 115.8)
- added U1: LM317_TO-220, Package_TO_SOT_THT:TO-220-3_Vertical, F.Cu at (157.7, 49.7)
- added U2: LM337_TO220, Package_TO_SOT_THT:TO-220-3_Vertical, F.Cu at (162.8, 122.7)
- C10, C9: value 4700u -> 10u; footprint Capacitor_THT:CP_Radial_D18.0mm_P7.50mm -> Capacitor_THT:CP_Radial_D4.0mm_P2.00mm
- moved C9 26.8 mm to (149.3, 66.0), turned to 180 degrees
- moved C12 11.7 mm to (135.4, 121.1)
- moved C10 11.6 mm to (147.1, 106.7), turned to 0 degrees
- moved C11 11.0 mm to (135.1, 59.4)
- moved J1 2.03 mm to (82.3, 105.7)
- moved C2 0.51 mm to (114.3, 93.1)
- moved J3 0.51 mm to (171.2, 86.4)
- moved J3 0.51 mm to (164.7, 86.4)
- moved J7 0.51 mm to (185.0, 88.9)
Connections:
- C1 pad 1: /V+ -> /UNREG+
- C10 pad 2: /V- -> Net-(U2-ADJ)
- C11 pad 1: /V+ -> /UNREG+
- C12 pad 2: /V- -> /UNREG-
- C2 pad 2: /V- -> /UNREG-
- C5 pad 1: /V+ -> /UNREG+
- C6 pad 2: /V- -> /UNREG-
- C7 pad 1: /V+ -> /UNREG+
- C8 pad 2: /V- -> /UNREG-
- C9 pad 1: /V+ -> Net-(U1-ADJ)
- D1 pad 1: /V+ -> /UNREG+
- D2 pad 2: /V- -> /UNREG-
- D3 pad 1: /V+ -> /UNREG+
- D4 pad 2: /V- -> /UNREG-
Routing:
- net GND: track 111.4 -> 175.3 mm
- net /V-: track 0.00 -> 58.7 mm
- net /V+: track 0.00 -> 43.6 mm
- net /UNREG+: track 0.00 -> 32.2 mm
- net /UNREG-: track 0.00 -> 32.2 mm
- net Net-(Q2-B): track 0.00 -> 31.0 mm
- net Net-(U2-ADJ): track 0.00 -> 30.3 mm
- net Net-(U1-ADJ): track 0.00 -> 27.4 mm
- net Net-(Q1-B): track 0.00 -> 12.0 mm
- net /AC2: track 29.8 -> 34.9 mm
- net /AC1: track 35.6 -> 38.6 mm
- added copper zone on B.Cu, net /UNREG+
- added copper zone on B.Cu, net /UNREG-
Other:
- board text added: "AC1"
- board text added: "AC2"
- board text added: "CT"
- board text removed: "AC"
