File: kicad/power_supply/power_supply.kicad_sch (KiCad schematic)
At the start: 23 parts, among them J1 AC1, J2 GND, J3 CT, J4 AC2, J5 V-, J6 V+, J7 GND

Commit message: Preparing for public release
Parts:
- removed C3, C4: 100n, Capacitor_THT:C_Rect_L7.2mm_W5.5mm_P5.00mm_FKS2_FKP2_MKS2_MKP2, symbol Device:C
- added C13, C14: 4700u, Capacitor_THT:CP_Radial_D18.0mm_P7.50mm, symbol Device:C_Polarized
- added H1, H2, H3, H4: MountingHole, MountingHole:MountingHole_3.2mm_M3, symbol Mechanical:MountingHole
- added Q1: TIP147, Package_TO_SOT_THT:TO-247-3_Horizontal_TabDown, symbol Transistor_BJT:TIP127
- added Q2: TIP142, Package_TO_SOT_THT:TO-247-3_Horizontal_TabDown, symbol Transistor_BJT:TIP121
- added R1, R3: 22, Resistor_THT:R_Axial_DIN0204_L3.6mm_D1.6mm_P7.62mm_Horizontal, symbol Device:R
- added R2, R4: 150, Resistor_THT:R_Axial_DIN0204_L3.6mm_D1.6mm_P7.62mm_Horizontal, symbol Device:R
- added RV1, RV2: 2k, Custom:TRIM_T93YA103KT20, symbol Device:R_Potentiometer_Trim
- added U1: LM317_TO-220, Package_TO_SOT_THT:TO-220-3_Vertical, symbol Regulator_Linear:LM317_TO-220
- added U2: LM337_TO220, Package_TO_SOT_THT:TO-220-3_Vertical, symbol Regulator_Linear:LM337_TO220
- C10, C9: value 4700u -> 10u; footprint Capacitor_THT:CP_Radial_D18.0mm_P7.50mm -> Capacitor_THT:CP_Radial_D4.0mm_P2.00mm
Connections:
- net GND: now also C13.2, C14.1, RV1.2, RV1.3, RV2.1, RV2.2
- net V+: now also Q1.2 (C), R2.2, U1.2 (VO); no longer C1.1, C11.1, C5.1, C7.1, C9.1, D1.1 (K), D3.1 (K)
- net V-: now also Q2.2 (C), R4.1, U2.3 (VO); no longer C10.2, C12.2, C2.2, C6.2, C8.2, D2.2 (A), D4.2 (A)
- new net: Q1.1 (B), R1.2, U1.3 (VI)
- new net: C10.2, R4.2, RV2.3, U2.1 (ADJ)
- new net: C9.1, R2.1, RV1.1, U1.1 (ADJ)
- new net: Q2.1 (B), R3.2, U2.2 (VI)
- new net UNREG+: C1.1, C11.1, C13.1, C5.1, C7.1, D1.1 (K), D3.1 (K), Q1.3 (E), R1.1
- new net UNREG-: C12.2, C14.2, C2.2, C6.2, C8.2, D2.2 (A), D4.2 (A), Q2.3 (E), R3.1
Other:
- moved on the sheet: C1, C2, C5, C6, C7, C8, D1, D2, D3, D4, J1, J2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
