File: kicad/power_supply/power_supply.kicad_sch (KiCad schematic)
At the start: 37 parts, among them J1 AC1, J2 GND, J3 CT, J4 AC2, J5 V-, J6 V+, J7 GND, Q1 TIP147, Q2 TIP142, U1 LM317_TO-220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

Commit message: PCB improvments and lineup's adjustments.
Parts:
- R2, R4: value 150 -> 220
- RV1, RV2: value 2k -> 5k
Changed lines of the file:
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@@
 			)
 		)
-		(property "Value" "150"
+		(property "Value" "220"
 			(at 194.31 132.0799 0)
 			(effects
@@
 			)
 		)
-		(property "Value" "2k"
+		(property "Value" "5k"
 			(at 177.8 121.9199 0)
 			(effects
@@
 			)
 		)
-		(property "Value" "150"
+		(property "Value" "220"
 			(at 195.58 90.1699 0)
 			(effects
@@
 			)
 		)
-		(property "Value" "2k"
+		(property "Value" "5k"
 			(at 177.8 100.3299 0)
 			(effects
