File: kicad/power_supply/_autosave-power_supply.kicad_sch (KiCad schematic)
At the start: 37 parts, among them J1 AC1, J2 GND, J3 CT, J4 AC2, J5 V-, J6 V+, J7 GND, Q1 TIP147, Q2 TIP142, U1 LM317_TO-220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

Commit message: Restored after rebase mishap
Connections:
- net GND: now also C10.1, C9.2
- net V+: no longer C9.1
- net V-: no longer C10.2
- net at R4.2, RV2.3, U2.1 (ADJ): now also C10.2; no longer C10.1
- net at R2.1, RV1.1, U1.1 (ADJ): now also C9.1; no longer C9.2
Other:
- moved on the sheet: C10, C9
Changed lines of the file:
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@@
 	)
 	(junction
-		(at 129.54 110.49)
+		(at 204.47 110.49)
 		(diameter 0)
 		(color 0 0 0 0)
 	)
 	(junction
-		(at 163.83 83.82)
+		(at 129.54 110.49)
 		(diameter 0)
 		(color 0 0 0 0)
 	)
 	(junction
-		(at 129.54 125.73)
+		(at 163.83 83.82)
 		(diameter 0)
 		(color 0 0 0 0)
 	)
 	(junction
-		(at 204.47 153.67)
+		(at 129.54 125.73)
 		(diameter 0)
 		(color 0 0 0 0)
@@
 	)
 	(junction
-		(at 204.47 71.12)
-		(diameter 0)
-		(color 0 0 0 0)
-	)
-	(junction
 		(at 73.66 125.73)
 		(diameter 0)
@@
 	(wire
 		(pts
+			(xy 204.47 110.49) (xy 213.36 110.49)
+		)
+		(stroke
+			(width 0)
+			(type default)
+		)
+	)
+	(wire
+		(pts
 			(xy 60.96 125.73) (xy 60.96 121.92)
 		)
@@
 	(wire
 		(pts
+			(xy 204.47 110.49) (xy 204.47 114.3)
+		)
+		(stroke
+			(width 0)
+			(type default)
+		)
+	)
+	(wire
+		(pts
 			(xy 49.53 107.95) (xy 73.66 107.95)
 		)
@@
 	(wire
 		(pts
-			(xy 193.04 71.12) (xy 204.47 71.12)
+			(xy 193.04 71.12) (xy 213.36 71.12)
 		)
 		(stroke
@@
 	(wire
 		(pts
-			(xy 204.47 71.12) (xy 204.47 85.09)
-		)
-		(stroke
-			(width 0)
-			(type default)
-		)
-	)
-	(wire
-		(pts
-			(xy 204.47 135.89) (xy 204.47 153.67)
+			(xy 204.47 93.98) (xy 204.47 99.06)
 		)
 		(stroke
@@
 	(wire
 		(pts
-			(xy 185.42 110.49) (xy 213.36 110.49)
+			(xy 185.42 110.49) (xy 204.47 110.49)
 		)
 		(stroke
@@
 	(wire
 		(pts
+			(xy 204.47 121.92) (xy 204.47 125.73)
+		)
+		(stroke
+			(width 0)
+			(type default)
+		)
+	)
+	(wire
+		(pts
 			(xy 60.96 106.68) (xy 60.96 113.03)
 		)
@@
 	(wire
 		(pts
-			(xy 204.47 153.67) (xy 213.36 153.67)
+			(xy 191.77 153.67) (xy 213.36 153.67)
 		)
 		(stroke
@@
 	(wire
 		(pts
-			(xy 204.47 92.71) (xy 204.47 93.98)
-		)
-		(stroke
-			(width 0)
-			(type default)
-		)
-	)
-	(wire
-		(pts
 			(xy 87.63 125.73) (xy 73.66 125.73)
 		)
@@
 	(wire
 		(pts
-			(xy 191.77 153.67) (xy 204.47 153.67)
-		)
-		(stroke
-			(width 0)
-			(type default)
-		)
-	)
-	(wire
-		(pts
 			(xy 142.24 121.92) (xy 142.24 125.73)
 		)
@@
 	(wire
 		(pts
-			(xy 60.96 95.25) (xy 73.66 95.25)
+			(xy 204.47 106.68) (xy 204.47 110.49)
 		)
 		(stroke
@@
 	(wire
 		(pts
-			(xy 116.84 125.73) (xy 129.54 125.73)
+			(xy 60.96 95.25) (xy 73.66 95.25)
 		)
 		(stroke
@@
 	(wire
 		(pts
-			(xy 180.34 93.98) (xy 180.34 95.25)
+			(xy 116.84 125.73) (xy 129.54 125.73)
 		)
 		(stroke
@@
 	(wire
 		(pts
-			(xy 102.87 106.68) (xy 102.87 110.49)
+			(xy 180.34 93.98) (xy 180.34 95.25)
 		)
 		(stroke
@@
 	(wire
 		(pts
-			(xy 204.47 71.12) (xy 213.36 71.12)
+			(xy 102.87 106.68) (xy 102.87 110.49)
 		)
 		(stroke
@@
 		)
 	)
-	(wire
-		(pts
-			(xy 204.47 128.27) (xy 204.47 125.73)
-		)
-		(stroke
-			(width 0)
-			(type default)
-		)
-	)
 	(label "AC1"
 		(at 55.88 107.95 0)
@@
 	(symbol
 		(lib_id "Device:C_Polarized")
-		(at 204.47 132.08 0)
+		(at 204.47 118.11 0)
 		(unit 1)
 		(exclude_from_sim no)
@@
 		(fields_autoplaced yes)
 		(property "Reference" "C10"
-			(at 208.28 129.9209 0)
+			(at 208.28 115.9509 0)
 			(effects
 				(font
@@
 		)
 		(property "Value" "10u"
-			(at 208.28 132.4609 0)
+			(at 208.28 118.4909 0)
 			(effects
 				(font
@@
 		)
 		(property "Footprint" "Capacitor_THT:CP_Radial_D4.0mm_P2.00mm"
-			(at 205.4352 135.89 0)
+			(at 205.4352 121.92 0)
 			(effects
 				(font
@@
 		)
 		(property "Datasheet" "~"
-			(at 204.47 132.08 0)
+			(at 204.47 118.11 0)
 			(effects
 				(font
@@
 		)
 		(property "Description" "Polarized capacitor"
-			(at 204.47 132.08 0)
+			(at 204.47 118.11 0)
 			(effects
 				(font
@@
 	(symbol
 		(lib_id "Device:C_Polarized")
-		(at 204.47 88.9 0)
+		(at 204.47 102.87 0)
 		(unit 1)
 		(exclude_from_sim no)
@@
 		(fields_autoplaced yes)
 		(property "Reference" "C9"
-			(at 208.28 86.7409 0)
+			(at 208.28 100.7109 0)
 			(effects
 				(font
@@
 		)
 		(property "Value" "10u"
-			(at 208.28 89.2809 0)
+			(at 208.28 103.2509 0)
 			(effects
 				(font
@@
 		)
 		(property "Footprint" "Capacitor_THT:CP_Radial_D4.0mm_P2.00mm"
-			(at 205.4352 92.71 0)
+			(at 205.4352 106.68 0)
 			(effects
 				(font
@@
 		)
 		(property "Datasheet" "~"
-			(at 204.47 88.9 0)
+			(at 204.47 102.87 0)
 			(effects
 				(font
@@
 		)
 		(property "Description" "Polarized capacitor"
-			(at 204.47 88.9 0)
+			(at 204.47 102.87 0)
 			(effects
 				(font
